Commit message: built rb1 urdf replica - fix included

File: my_rb1_description/urdf/my_rb1_robot.urdf (robot description, URDF)
Before this commit: robot my_rb1_robot, 7 links, 6 joints
Links:
- link front_laser: geometry collision cylinder length=0.02 radius=0.03; visual cylinder length=0.02 radius=0.03
Joints:
- joint joint_back_caster: type continuous -> fixed
- joint joint_front_caster: type continuous -> fixed
